Commit message: modified xacro files to add colors for the components

File: agv_low/robots/agv_urdf.xacro (robot description, xacro)
@@ -11,4 +11,6 @@
 	<!-- Import all available sensors -->
 	<xacro:include filename="$(find agv_low)/urdf/sensors/all_sensors.urdf.xacro" />
+	<!-- Import all colors -->
+	<xacro:include filename="$(find agv_low)/urdf/materials.xacro" />
 	<xacro:arg name="prefix" default="agv_"/>
     	<xacro:macro name="agv" params="prefix">
@@ -24,5 +26,4 @@
   		<xacro:mecanum_wheel prefix="${prefix}back_right" angle="1" wheel_pos="1" parent="${prefix}base_link" />
   		<!-- IMU -->
-<!--
 		<xacro:sensor_imu_hector prefix="$(arg prefix)imu" parent="$(arg prefix)base_link">
 			<origin xyz="0.48 0.0 0.338" rpy="0 0 0"/>
@@ -34,13 +35,12 @@
 			<origin xyz="0.060 -0.349 0.338" rpy="0 0 3.1416"/>
 		</xacro:sensor_sick_s300>
-		<xacro:sensor_asus_xtion_pro prefix="$(arg prefix)xtion" parent="$(arg prefix)base_link" > -->
+		<xacro:sensor_asus_xtion_pro prefix="$(arg prefix)xtion" parent="$(arg prefix)base_link" >
 			<!--<origin xyz="0.900 -0.0235 0.338" rpy="0 0 0" /> -->
-<!--			<origin xyz="0.900 -0.0235 0.35075" rpy="0 1.571 -3.1416" />
+			<origin xyz="0.900 -0.0235 0.35075" rpy="0 1.571 -3.1416" />
 		</xacro:sensor_asus_xtion_pro>
-		<xacro:sensor_asus_xtion_pro_stand prefix="$(arg prefix)xtion_stand" parent="$(arg prefix)base_link" > -->
+		<xacro:sensor_asus_xtion_pro_stand prefix="$(arg prefix)xtion_stand" parent="$(arg prefix)base_link" >
 			<!--<origin xyz="0.900 -0.0235 0.338" rpy="0 0 0" /> -->
-<!--			<origin xyz="0.900 -0.0235 0.338" rpy="0 0 0" />
+			<origin xyz="0.900 -0.0235 0.338" rpy="0 0 0" />
 		</xacro:sensor_asus_xtion_pro_stand>
-		-->
    	</xacro:macro>
    <!-- Gazebo ros control pluggins -->

File: agv_low/urdf/bases/agv_low_base_gazebo_urdf.xacro (robot description, xacro)
@@ -46,6 +46,6 @@
 		<gazebo>
 	    <plugin name="planar_move" filename="libgazebo_ros_planar_move.so">
-	      <commandTopic>agv/cmd_vel</commandTopic>
-	      <odometryTopic>agv/odom</odometryTopic>
+	      <commandTopic>cmd_vel</commandTopic>
+	      <odometryTopic>odom</odometryTopic>
 	      <odometryFrame>${prefix}odom</odometryFrame>
 	      <odometryRate>50.0</odometryRate>

File: agv_low/urdf/bases/agv_low_base_urdf.xacro (robot description, xacro)
@@ -27,4 +27,5 @@
 				<mesh filename="package://agv_low/meshes/Plattform Baugruppe_20171217_WO_wheels_collision_as_original.stl"/>
 			</geometry>
+			<material name="white"/>
 		</visual>
 		<collision>

File: agv_low/urdf/sensors/asus_xtion_pro_stand.xacro (robot description, xacro)
@@ -7,17 +7,4 @@
   <xacro:property name="asus_xtion_scale" value="1.0"/>
   <xacro:macro name="sensor_asus_xtion_pro_stand" params="prefix parent *origin">
-<!--   <joint name="${prefix}_stand_footprint_joint" type ="fixed">
-    <xacro:insert_block name="origin" />
-    <parent link="${parent}"/>
-    <child link="${prefix}_stand_footprint"/>
-   </joint>
-   <link name="${prefix}_stand_footprint">
-    <visual>
-     <origin xyz="0 0 0" rpy="0 0 0" />
-     <geometry>
-      <box size="0.001 0.001 0.001" />
-     </geometry>
-    </visual>
-   </link> -->
    <joint name="${prefix}_stand_joint" type ="fixed">
     <xacro:insert_block name="origin" />
@@ -30,6 +17,7 @@
 		<origin xyz="0 0 0" rpy="${M_PI/2} 0 ${M_PI/2}"/>
         <geometry>
-          <mesh filename="package://agv_low/meshes/sensors/base_new.dae" scale="${asus_xtion_scale} ${asus_xtion_scale} ${asus_xtion_scale}"/>
+          <mesh filename="package://agv_low/meshes/sensors/base_new.stl" scale="${asus_xtion_scale} ${asus_xtion_scale} ${asus_xtion_scale}"/>
         </geometry>
+	<material name="black"/>
       </visual>
       <collision>
@@ -48,4 +36,8 @@
       </inertial>
     </link>
+    <gazebo reference = "${prefix}_base">
+     <material>Gazebo/Black</material>
+     <turnGravityOff>false</turnGravityOff>
+    </gazebo>
   </xacro:macro>
 </robot>

File: agv_low/urdf/wheels/agv_low_wheel_urdf.xacro (robot description, xacro)
@@ -40,5 +40,6 @@
               <mesh filename="package://agv_low/meshes/Radbefestigung mit Motor-Getrieb (LVA33)_MIR_wheels.stl" />
             </geometry>
-	  </xacro:unless>
+			 </xacro:unless>
+	  	   <material name="grey"/>
       </visual>
       <collision>
@@ -54,5 +55,5 @@
       </inertial>
     </link>
-    <!-- Transmission is important to link the joints and the controller (see summit_xl_control/config/summit_xl_control.yaml)-->
+    <!-- Transmission is important to link the joints and the controller-->
     <transmission name="${prefix}_wheel_joint_trans">
       <type>transmission_interface/SimpleTransmission</type>
@@ -70,9 +71,6 @@
 		<kd value="1.0" />
 		<fdir1 value="1 0 0"/>
-        <turnGravityOff>false</turnGravityOff>
-    </gazebo>
-    <gazebo reference="${prefix}base_link">
-     <material>Gazebo/Black</material>
-     <turnGravityOff>false</turnGravityOff>
+		<material>Gazebo/Grey</material>
+      <turnGravityOff>false</turnGravityOff>
     </gazebo>
   </xacro:macro>

Commit message: changed collision elements in urdf to solids and commented the sensors in launch file

File: agv_low/robots/agv_urdf.xacro (robot description, xacro)
@@ -21,9 +21,12 @@
 		<!-- Summit XL base -->
 		<xacro:agv_base prefix="$(arg prefix)" />
+<!--
 		<xacro:mecanum_wheel prefix="${prefix}front_left" angle="-1" wheel_pos="1" parent="${prefix}base_link" />
   		<xacro:mecanum_wheel prefix="${prefix}front_right" angle="1" wheel_pos="-1" parent="${prefix}base_link" />
   		<xacro:mecanum_wheel prefix="${prefix}back_left" angle="-1" wheel_pos="-1" parent="${prefix}base_link" />
   		<xacro:mecanum_wheel prefix="${prefix}back_right" angle="1" wheel_pos="1" parent="${prefix}base_link" />
+-->
   		<!-- IMU -->
+<!--
 		<xacro:sensor_imu_hector prefix="$(arg prefix)imu" parent="$(arg prefix)base_link">
 			<origin xyz="0.48 0.0 0.338" rpy="0 0 0"/>
@@ -35,13 +38,14 @@
 			<origin xyz="0.060 -0.349 0.338" rpy="0 0 3.1416"/>
 		</xacro:sensor_sick_s300>
-		<xacro:sensor_asus_xtion_pro prefix="$(arg prefix)xtion" parent="$(arg prefix)base_link" >
+		<xacro:sensor_asus_xtion_pro prefix="$(arg prefix)xtion" parent="$(arg prefix)base_link" > -->
 			<!--<origin xyz="0.900 -0.0235 0.338" rpy="0 0 0" /> -->
 			<!--<origin xyz="0.900 -0.0235 0.35075" rpy="0 1.571 -3.1416" /> 0.37225 -->
-			<origin xyz="0.87852 -0.0015 0.36875" rpy="0 -1.571 0" />
+<!--			<origin xyz="0.87852 -0.0015 0.36875" rpy="0 -1.571 0" />
 		</xacro:sensor_asus_xtion_pro>
-		<xacro:sensor_asus_xtion_pro_stand prefix="$(arg prefix)xtion_stand" parent="$(arg prefix)base_link" >
+		<xacro:sensor_asus_xtion_pro_stand prefix="$(arg prefix)xtion_stand" parent="$(arg prefix)base_link" > -->
 			<!--<origin xyz="0.900 -0.0235 0.338" rpy="0 0 0" /> -->
-			<origin xyz="0.900 -0.0235 0.338" rpy="0 0 0" />
+<!--			<origin xyz="0.900 -0.0235 0.338" rpy="0 0 0" />
 		</xacro:sensor_asus_xtion_pro_stand>
+-->
    	</xacro:macro>
    <!-- Gazebo ros control pluggins -->

File: agv_low/robots/agv_urdf_youbot_collsionwheel.xacro (robot description, xacro)
@@ -34,4 +34,5 @@
   		<xacro:mecanum_wheel_visual prefix="${prefix}back_right" angle="1" wheel_pos="1" parent="${prefix}base_link" />
   		<!-- IMU -->
+<!--
 		<xacro:sensor_imu_hector prefix="$(arg prefix)imu" parent="$(arg prefix)base_link">
 			<origin xyz="0.48 0.0 0.338" rpy="0 0 0"/>
@@ -43,12 +44,13 @@
 			<origin xyz="0.060 -0.349 0.338" rpy="0 0 3.1416"/>
 		</xacro:sensor_sick_s300>
-		<xacro:sensor_asus_xtion_pro prefix="$(arg prefix)xtion" parent="$(arg prefix)base_link" >
+		<xacro:sensor_asus_xtion_pro prefix="$(arg prefix)xtion" parent="$(arg prefix)base_link" > -->
 			<!--<origin xyz="0.900 -0.0235 0.338" rpy="0 0 0" /> -->
-			<origin xyz="0.87852 -0.0015 0.36875" rpy="0 -1.571 0" />
+<!--			<origin xyz="0.87852 -0.0015 0.36875" rpy="0 -1.571 0" />
 		</xacro:sensor_asus_xtion_pro>
-		<xacro:sensor_asus_xtion_pro_stand prefix="$(arg prefix)xtion_stand" parent="$(arg prefix)base_link" >
+		<xacro:sensor_asus_xtion_pro_stand prefix="$(arg prefix)xtion_stand" parent="$(arg prefix)base_link" > -->
 			<!--<origin xyz="0.900 -0.0235 0.338" rpy="0 0 0" /> -->
-			<origin xyz="0.900 -0.0235 0.338" rpy="0 0 0" />
+<!--			<origin xyz="0.900 -0.0235 0.338" rpy="0 0 0" />
 		</xacro:sensor_asus_xtion_pro_stand>
+-->
    	</xacro:macro>
    <!-- Gazebo ros control pluggins -->

File: agv_low/urdf/bases/agv_low_base_urdf.xacro (robot description, xacro)
@@ -23,5 +23,5 @@
   		</inertial>
 		<visual>
-			<origin xyz="0 0 0.308" rpy="-1.57 0 0"/>
+			<origin xyz="0 0 0.308" rpy="-1.57 0 0"/> <!-- xyz="0 0 0.308" rpy="-1.57 0 0" -->
 			<geometry>
 				<mesh filename="package://agv_low/meshes/Plattform Baugruppe_20171217_WO_wheels_collision_as_original.stl"/>
@@ -30,7 +30,7 @@
 		</visual>
 		<collision>
-			<origin xyz="0 0 0.308" rpy="-1.57 0 0"/>
+			<origin xyz="0.48 -0.0235 0.188" rpy="0 0 0"/>
 			<geometry>
-				<mesh filename="package://agv_low/meshes/Plattform Baugruppe_20171217_WO_wheels_collision_as_original.stl"/>
+				<box size="1.020 0.763 0.300"/> <!-- 1.020 0.763 0.300 -->
 			</geometry>
 		</collision>

File: agv_low/urdf/wheels/agv_low_wheel_urdf_visualwheel.xacro (robot description, xacro)
@@ -1,10 +1,10 @@
 <?xml version="1.0" encoding="UTF-8"?>
 <robot name="wheel" xmlns:xacro="http://www.ros.org/wiki/xacro">
-  <xacro:property name="wheel_mass" value="2.166" /> <!-- in kg-->
+  <xacro:property name="wheel_mass" value="0.1" /> <!-- 2.166 in kg-->
   <xacro:property name="pi" value="3.14159"/>
   <xacro:macro name="mecanum_inertia">
-    <inertia  ixx="0.008" ixy = "0" ixz = "0"
-              iyy="0.008" iyz = "0"
-              izz="0.010" />
+    <inertia  ixx="0.000" ixy = "0" ixz = "0"
+              iyy="0.000" iyz = "0"
+              izz="0.000" />
   </xacro:macro>
   <xacro:macro name="mecanum_wheel_visual" params="prefix angle wheel_pos parent">
@@ -53,5 +53,5 @@
 		<mu2 value="1.0"/>
 		<kp value="10000000.0" />
-		<kd value="1.0" />
+		<kd value="100.0" />
 		<fdir1 value="1 0 0"/>
 		<material>Gazebo/Grey</material>

File: agv_low/urdf/wheels/agv_low_wheel_urdf_youbot_collision.xacro (robot description, xacro)
@@ -61,5 +61,6 @@
 	<origin xyz="0 0 0" rpy="${pi*angle/2} 0 0" />
         <geometry>
-	  <mesh filename="package://agv_low/meshes/agv_sphere_wheel.stl"/>
+	 <sphere radius="0.103"/>
+<!--	  <mesh filename="package://agv_low/meshes/agv_sphere_wheel.stl"/> -->
 	</geometry>
       </collision>
@@ -67,4 +68,5 @@
 	<origin xyz="0 0 0" rpy="${pi*angle/2} 0 0" />
         <geometry>
+	 <sphere radius="0.103"/>
 	  <mesh filename="package://agv_low/meshes/agv_sphere_wheel.stl"/>
 	</geometry>
