Commit message: mecanum wheel simulation

File: agv_low/robots/agv_urdf_collsionwheel.xacro (robot description, xacro)
@@ -7,7 +7,6 @@
 	<!-- Import summit XL base elements -->
 	<xacro:include filename="$(find agv_low)/urdf/bases/agv_low_base_urdf.xacro" />
-	<xacro:include filename="$(find agv_low)/urdf/bases/agv_low_base_gazebo_urdf.xacro" />
 	<!-- Import summit XL wheels collision -->
-	<xacro:include filename="$(find agv_low)/urdf/wheels/agv_low_wheel_urdf_youbot_collision.xacro" />
+	<xacro:include filename="$(find agv_low)/urdf/wheels/agv_low_wheel_urdf_collisionwheel.xacro" />
 	<!-- Import summit XL wheels visual -->
 	<xacro:include filename="$(find agv_low)/urdf/wheels/agv_low_wheel_urdf_visualwheel.xacro" />
@@ -16,6 +15,4 @@
 	<!-- Import all colors -->
 	<xacro:include filename="$(find agv_low)/urdf/materials.xacro" />
-	<!-- ros controller -->
-        <xacro:include filename="$(find agv_low)/urdf/ros_controller.urdf.xacro" />
 	<xacro:arg name="prefix" default="agv_"/>
     	<xacro:macro name="agv" params="prefix">
@@ -26,39 +23,37 @@
 		<!-- Summit XL base -->
 		<xacro:agv_base prefix="$(arg prefix)" />
-		<xacro:mecanum_wheel_youbot_collision prefix="${prefix}front_left" angle="-1" parent="${prefix}base_link" />
-  		<xacro:mecanum_wheel_youbot_collision prefix="${prefix}front_right" angle="1" parent="${prefix}base_link" />
-  		<xacro:mecanum_wheel_youbot_collision prefix="${prefix}back_left" angle="-1" parent="${prefix}base_link" />
-  		<xacro:mecanum_wheel_youbot_collision prefix="${prefix}back_right" angle="1" parent="${prefix}base_link" />
-		<xacro:mecanum_wheel_visual prefix="${prefix}front_left" angle="-1" wheel_pos="0" parent="${prefix}base_link" />
-  		<xacro:mecanum_wheel_visual prefix="${prefix}front_right" angle="1" wheel_pos="1" parent="${prefix}base_link" />
-  		<xacro:mecanum_wheel_visual prefix="${prefix}back_left" angle="-1" wheel_pos="1" parent="${prefix}base_link" />
-  		<xacro:mecanum_wheel_visual prefix="${prefix}back_right" angle="1" wheel_pos="0" parent="${prefix}base_link" />
-		<!-- Gazebo ros control pluggins -->
+		<xacro:mecanum_wheel_collision prefix="${prefix}front_left" angle="-1" wheel_pos="1" parent="${prefix}base_link" />
+  		<xacro:mecanum_wheel_collision prefix="${prefix}front_right" angle="1" wheel_pos="-1" parent="${prefix}base_link" />
+  		<xacro:mecanum_wheel_collision prefix="${prefix}back_left" angle="-1" wheel_pos="-1" parent="${prefix}base_link" />
+  		<xacro:mecanum_wheel_collision prefix="${prefix}back_right" angle="1" wheel_pos="1" parent="${prefix}base_link" />
+		<xacro:mecanum_wheel_visual prefix="${prefix}front_left" angle="-1" wheel_pos="1" parent="${prefix}base_link" />
+  		<xacro:mecanum_wheel_visual prefix="${prefix}front_right" angle="1" wheel_pos="-1" parent="${prefix}base_link" />
+  		<xacro:mecanum_wheel_visual prefix="${prefix}back_left" angle="-1" wheel_pos="-1" parent="${prefix}base_link" />
+  		<xacro:mecanum_wheel_visual prefix="${prefix}back_right" angle="1" wheel_pos="1" parent="${prefix}base_link" />
   		<!-- IMU -->
 <!--
 		<xacro:sensor_imu_hector prefix="$(arg prefix)imu" parent="$(arg prefix)base_link">
-			<origin xyz="0.0 0.0 0.0" rpy="0 0 0"/>
+			<origin xyz="0.48 0.0 0.338" rpy="0 0 0"/>
 		</xacro:sensor_imu_hector>
 		<xacro:sensor_sick_s300 prefix="$(arg prefix)s300_front" parent="$(arg prefix)base_link" prefix_topic="front_laser">
-			<origin xyz="0.41 0.320 0.0" rpy="0 0 0"/>
+			<origin xyz="0.900 0.300 0.338" rpy="0 0 0"/>
 		</xacro:sensor_sick_s300>
 		<xacro:sensor_sick_s300 prefix="$(arg prefix)s300_back" parent="$(arg prefix)base_link" prefix_topic="back_laser">
-			<origin xyz="-0.41 -0.320 0.0" rpy="0 0 3.1416"/>
+			<origin xyz="0.060 -0.349 0.338" rpy="0 0 3.1416"/>
 		</xacro:sensor_sick_s300>
 		<xacro:sensor_asus_xtion_pro prefix="$(arg prefix)xtion" parent="$(arg prefix)base_link" > -->
 			<!--<origin xyz="0.900 -0.0235 0.338" rpy="0 0 0" /> -->
-<!--			<origin xyz="0.39852 -0.0015 0.36875" rpy="0 -1.571 0" />
+<!--			<origin xyz="0.900 -0.0235 0.35075" rpy="0 1.571 -3.1416" />
 		</xacro:sensor_asus_xtion_pro>
 		<xacro:sensor_asus_xtion_pro_stand prefix="$(arg prefix)xtion_stand" parent="$(arg prefix)base_link" > -->
 			<!--<origin xyz="0.900 -0.0235 0.338" rpy="0 0 0" /> -->
-<!--			<origin xyz="0.42 -0.0235 0.0" rpy="0 0 0" />
+<!--			<origin xyz="0.900 -0.0235 0.338" rpy="0 0 0" />
 		</xacro:sensor_asus_xtion_pro_stand>
--->
+ -->
    	</xacro:macro>
    <!-- Gazebo ros control pluggins -->
-<!--    <xacro:ros_control />  -->
+   <!-- <xacro:ros_control /> -->
    <!-- <xacro:ros_force_based_move prefix="$(arg prefix)"/> -->
 <!--   <xacro:planar_move prefix="$(arg prefix)"/> -->
-   <xacro:fourwheel_visual_diff_drive prefix="$(arg prefix)"/>
    <xacro:agv prefix="$(arg prefix)"/>
    <!--<xacro:xtion_stand parent="agv_base_link" tilting_angle="0" /> -->

File: agv_low/urdf/bases/agv_low_base_gazebo_urdf.xacro (robot description, xacro)
@@ -6,6 +6,6 @@
       <plugin name="ros_control" filename="libgazebo_ros_control.so">
         <!--<robotNamespace>/agv_low</robotNamespace>-->
-	<robotParam>robot_description</robotParam>
-        <controlPeriod>0.001</controlPeriod>
+<!--	<robotParam>robot_description</robotParam>
+        <controlPeriod>0.001</controlPeriod> -->
 	<robotSimType>gazebo_ros_control/DefaultRobotHWSim</robotSimType>
       </plugin>
@@ -55,3 +55,44 @@
 	  </gazebo>
   </xacro:macro>
+  <xacro:macro name="fourwheel_visual_diff_drive" params="prefix">
+   	<gazebo>
+  		<plugin name="fourwheel_visual_diff_drive_controller" filename="libfourwheel_drive_visual_wheel.so">
+   			<alwaysOn>true</alwaysOn>
+    			<updateRate>10</updateRate>
+    			<frontleftJoint>${prefix}front_left_wheel_joint_visual</frontleftJoint>
+    			<frontrightJoint>${prefix}front_right_wheel_joint_visual</frontrightJoint>
+    			<backleftJoint>${prefix}back_left_wheel_joint_visual</backleftJoint>
+    			<backrightJoint>${prefix}back_right_wheel_joint_visual</backrightJoint>
+    			<wheelDiameter>0.206</wheelDiameter>
+    			<wheelTorque>20</wheelTorque>
+   			<commandTopic>cmd_vel</commandTopic>
+<!--
+   			<odometryTopic>odom</odometryTopic>
+   			<odometryFrame>odom</odometryFrame>
+-->
+   			<robotBaseFrame>agv_base_footprint</robotBaseFrame>
+<!--   			<robotNamespace>gz</robotNamespace> -->
+   		</plugin>
+   	</gazebo>
+  </xacro:macro>
+<!--
+  <xacro:macro name="fourwheel_visual_diff_drive" params="prefix">
+   	<gazebo>
+  		<plugin name="differential_drive_controller" filename="libgazebo_ros_diff_drive.so">
+			<legacyMode>true</legacyMode>
+			<alwaysOn>true</alwaysOn>
+    			<updateRate>10</updateRate>
+    			<leftJoint>${prefix}front_left_wheel_joint_visual</leftJoint>
+    			<rightJoint>${prefix}front_right_wheel_joint_visual</rightJoint>
+			<wheelSeparation>0.6</wheelSeparation>
+    			<wheelDiameter>0.206</wheelDiameter>
+    			<torque>20</torque>
+   			<commandTopic>cmd_vel</commandTopic>
+   			<odometryTopic>odom</odometryTopic>
+   			<odometryFrame>odom</odometryFrame>
+   			<robotBaseFrame>agv_base_footprint</robotBaseFrame>
+   		</plugin>
+   	</gazebo>
+  </xacro:macro>
+-->
 </robot>

File: agv_low/urdf/bases/agv_low_base_urdf.xacro (robot description, xacro)
@@ -5,5 +5,5 @@
 	<link name="${prefix}base_footprint">
 		<visual>
-			<origin xyz="0 0 0" rpy="0 0 0" />
+			<origin xyz="0 0 0" rpy="0 0 0" /> <!-- "0.48 -0.0245 0.27" -->
 			<geometry>
 				<box size="0.001 0.001 0.001" />
@@ -12,23 +12,29 @@
 	</link>
 	<joint name="${prefix}base_footprint_joint" type="fixed">
-		<origin xyz="0 0 0" rpy="0 0 0" />
+		<origin xyz="0 0 0.338" rpy="0 0 0" /> <!-- "0.48 -0.0245 0" -->
 		<parent link="${prefix}base_footprint"/>
 		<child link="${prefix}base_link" />
 	</joint>
 	<link name="${prefix}base_link">
-		<inertial>
+<!--		<inertial>
     			<origin rpy="0 0 0" xyz="0.483 0.135 -0.025"/>
     			<mass value="39.096"/>
     			<inertia ixx="2.379" ixy="0.005" ixz="0" iyy="4.190" iyz="-0.001" izz="2.553"/>
   		</inertial>
+-->
+		<inertial>
+    			<origin rpy="0 0 0" xyz="0 0 0"/>
+    			<mass value="40.0"/>
+    			<inertia ixx="1.167" ixy="0.0" ixz="0.0" iyy="2.808" iyz="0.0" izz="2.241"/>
+  		</inertial>
 		<visual>
-			<origin xyz="0 0 0.308" rpy="-1.57 0 0"/> <!-- xyz="0 0 0.308" rpy="-1.57 0 0" -->
+			<origin xyz="0 0 0" rpy="0 0 0"/> <!-- xyz="0 0 0.338" -->
 			<geometry>
-				<mesh filename="package://agv_low/meshes/Plattform Baugruppe_20171217_WO_wheels_collision_as_original.stl"/>
+				<mesh filename="package://agv_low/meshes/Plattform Baugruppe_20171217_WO_wheels_collision_as_original_newxyz.stl"/>
 			</geometry>
 			<material name="white"/>
 		</visual>
 		<collision>
-			<origin xyz="0.48 -0.0235 0.188" rpy="0 0 0"/>
+			<origin xyz="0 0 -0.15" rpy="0 0 0"/> <!-- "0.48 -0.0235 0.188" -->
 			<geometry>
 				<box size="1.020 0.763 0.300"/> <!-- 1.020 0.763 0.300 -->

File: agv_low/urdf/ros_controller.urdf.xacro (robot description, xacro)
@@ -1,8 +1,7 @@
 <?xml version="1.0"?>
-<robot xmlns:sensor="http://playerstage.sourceforge.net/gazebo/xmlschema/#sensor"
-       xmlns:controller="http://playerstage.sourceforge.net/gazebo/xmlschema/#controller"
-       xmlns:interface="http://playerstage.sourceforge.net/gazebo/xmlschema/#interface">
+<robot xmlns:xacro="http://www.ros.org/wiki/xacro">
   <gazebo>
     <plugin name="gazebo_ros_controller" filename="libgazebo_ros_control.so" />
+    	<robotNamespace>agv_steeredwheel</robotNamespace>
   </gazebo>
 </robot>

File: agv_low/urdf/wheels/agv_low_wheel_urdf_visualwheel.xacro (robot description, xacro)
@@ -1,10 +1,16 @@
 <?xml version="1.0" encoding="UTF-8"?>
 <robot name="wheel" xmlns:xacro="http://www.ros.org/wiki/xacro">
-  <xacro:property name="wheel_mass" value="0.6" /> <!-- 2.166 in kg-->
+  <xacro:property name="wheel_mass" value="2" /> <!-- 2.166 in kg-->
   <xacro:property name="pi" value="3.14159"/>
+  <xacro:property name="wheel_joint_damping" value="1.0"/>
+  <xacro:property name="wheel_joint_friction" value="1.0"/>
+  <xacro:property name="wheel_joint_effort" value="30"/>
+  <xacro:property name="wheel_joint_velocity" value="10"/>
+  <xacro:property name="wheel_joint_safety_k_velocity" value="10.0"/>
+  <xacro:property name="wheel_mechanical_reduction" value="${624/35 * 80/18}" />
   <xacro:macro name="mecanum_inertia">
-    <inertia  ixx="1.5" ixy = "0" ixz = "0"
-              iyy="1.5" iyz = "0"
-              izz="1.5" />
+    <inertia  ixx="0.0085" ixy = "0" ixz = "0"
+              iyy="0.0085" iyz = "0"
+              izz="0.0085" />
   </xacro:macro>
   <xacro:macro name="mecanum_wheel_visual" params="prefix angle wheel_pos parent">
@@ -12,4 +18,5 @@
       <parent link="${parent}"/>
       <child link="${prefix}_wheel_link_visual"/>
+<!--
       <xacro:if value="${prefix == 'agv_front_left'}">
       	<origin xyz="0.835 0.213 0.103" />
@@ -24,7 +31,21 @@
       	<origin xyz="0.125 -0.262 0.102" />
       </xacro:if>
+-->
+      <xacro:if value="${prefix == 'agv_front_left'}">
+      	<origin xyz="0.355 0.237 -0.236" /> <!-- y = 0.213     0.355 0.237 -0.236 -->
+      </xacro:if>
+      <xacro:if value="${prefix == 'agv_front_right'}">
+      	<origin xyz="0.355 -0.237 -0.236" /> <!-- y = -0.261 -->
+      </xacro:if>
+      <xacro:if value="${prefix == 'agv_back_left'}">
+      	<origin xyz="-0.355 0.238 -0.236" /> <!-- y = 0.214 -->
+      </xacro:if>
+      <xacro:if value="${prefix == 'agv_back_right'}">
+      	<origin xyz="-0.355 -0.238 -0.236" /> <!-- y = -0.262 -->
+      </xacro:if>
       <axis xyz="0 1 0" rpy="0 0 0" />
-      <limit effort="100" velocity="100"/>
-      <joint_properties damping="0.0" friction="0.0"/>
+      <limit effort="${wheel_joint_effort}" velocity="${wheel_joint_velocity}"/>
+      <dynamics damping="${wheel_joint_damping}" friction="${wheel_joint_friction}"/>
+      <safety_controller k_velocity="${wheel_joint_safety_k_velocity}"/>
     </joint>
     <link name="${prefix}_wheel_link_visual">
@@ -41,17 +62,28 @@
             </geometry>
 	  </xacro:unless>
-	  <material name="grey"/>
       </visual>
       <inertial>
         <mass value="${wheel_mass}" />
-        <origin xyz="0 0 0.076" />
+        <origin xyz="0 0 0.076" /> <!-- "0 0 0.076" -->
         <xacro:mecanum_inertia />
       </inertial>
     </link>
+<!--
+    <transmission name="${prefix}_wheel_joint_visual_trans">
+      <type>transmission_interface/SimpleTransmission</type>
+      <actuator name="${prefix}_wheel_joint_visual_motor">
+        <hardwareInterface>hardware_interface/VelocityJointInterface</hardwareInterface>
+        <mechanicalReduction>${wheel_mechanical_reduction}</mechanicalReduction>
+      </actuator>
+      <joint name="${prefix}_wheel_joint_visual">
+        <hardwareInterface>hardware_interface/VelocityJointInterface</hardwareInterface>
+      </joint>
+    </transmission>
+-->
     <gazebo reference="${prefix}_wheel_link_visual">
 		<mu1 value="1.0"/>
 		<mu2 value="1.0"/>
 		<kp value="10000000.0" />
-		<kd value="100.0" />
+		<kd value="1.0" />
 		<fdir1 value="1 0 0"/>
 		<material>Gazebo/Grey</material>
