Commit message: created new urdf to simulate agv using youbot steered wheel plugin

File: agv_low/robots/agv_urdf_youbot_collsionwheel.xacro (robot description, xacro)
@@ -7,10 +7,14 @@
 	<!-- Import summit XL base elements -->
 	<xacro:include filename="$(find agv_low)/urdf/bases/agv_low_base_urdf.xacro" />
-	<!-- Import summit XL wheels -->
-	<xacro:include filename="$(find agv_low)/urdf/wheels/agv_low_wheel_urdf.xacro" />
+	<!-- Import summit XL wheels collision -->
+	<xacro:include filename="$(find agv_low)/urdf/wheels/agv_low_wheel_urdf_youbot_collision.xacro" />
+	<!-- Import summit XL wheels visual -->
+	<xacro:include filename="$(find agv_low)/urdf/wheels/agv_low_wheel_urdf_visualwheel.xacro" />
 	<!-- Import all available sensors -->
 	<xacro:include filename="$(find agv_low)/urdf/sensors/all_sensors.urdf.xacro" />
 	<!-- Import all colors -->
 	<xacro:include filename="$(find agv_low)/urdf/materials.xacro" />
+	<!-- ros controller -->
+        <xacro:include filename="$(find agv_low)/urdf/ros_controller.urdf.xacro" />
 	<xacro:arg name="prefix" default="agv_"/>
     	<xacro:macro name="agv" params="prefix">
@@ -21,8 +25,12 @@
 		<!-- Summit XL base -->
 		<xacro:agv_base prefix="$(arg prefix)" />
-		<xacro:mecanum_wheel prefix="${prefix}front_left" angle="-1" wheel_pos="1" parent="${prefix}base_link" />
-  		<xacro:mecanum_wheel prefix="${prefix}front_right" angle="1" wheel_pos="-1" parent="${prefix}base_link" />
-  		<xacro:mecanum_wheel prefix="${prefix}back_left" angle="-1" wheel_pos="-1" parent="${prefix}base_link" />
-  		<xacro:mecanum_wheel prefix="${prefix}back_right" angle="1" wheel_pos="1" parent="${prefix}base_link" />
+		<xacro:mecanum_wheel_youbot_collision prefix="${prefix}front_left" angle="-1" wheel_pos="1" parent="${prefix}base_link" />
+  		<xacro:mecanum_wheel_youbot_collision prefix="${prefix}front_right" angle="1" wheel_pos="-1" parent="${prefix}base_link" />
+  		<xacro:mecanum_wheel_youbot_collision prefix="${prefix}back_left" angle="-1" wheel_pos="-1" parent="${prefix}base_link" />
+  		<xacro:mecanum_wheel_youbot_collision prefix="${prefix}back_right" angle="1" wheel_pos="1" parent="${prefix}base_link" />
+		<xacro:mecanum_wheel_visual prefix="${prefix}front_left" angle="-1" wheel_pos="1" parent="${prefix}base_link" />
+  		<xacro:mecanum_wheel_visual prefix="${prefix}front_right" angle="1" wheel_pos="-1" parent="${prefix}base_link" />
+  		<xacro:mecanum_wheel_visual prefix="${prefix}back_left" angle="-1" wheel_pos="-1" parent="${prefix}base_link" />
+  		<xacro:mecanum_wheel_visual prefix="${prefix}back_right" angle="1" wheel_pos="1" parent="${prefix}base_link" />
   		<!-- IMU -->
 		<xacro:sensor_imu_hector prefix="$(arg prefix)imu" parent="$(arg prefix)base_link">
@@ -37,5 +45,4 @@
 		<xacro:sensor_asus_xtion_pro prefix="$(arg prefix)xtion" parent="$(arg prefix)base_link" >
 			<!--<origin xyz="0.900 -0.0235 0.338" rpy="0 0 0" /> -->
-			<!--<origin xyz="0.900 -0.0235 0.35075" rpy="0 1.571 -3.1416" /> 0.37225 -->
 			<origin xyz="0.87852 -0.0015 0.36875" rpy="0 -1.571 0" />
 		</xacro:sensor_asus_xtion_pro>
@@ -46,9 +53,7 @@
    	</xacro:macro>
    <!-- Gazebo ros control pluggins -->
-   <!-- <xacro:ros_control /> -->
+<!--    <xacro:ros_control /> -->
    <!-- <xacro:ros_force_based_move prefix="$(arg prefix)"/> -->
-<!--
-   <xacro:planar_move prefix="$(arg prefix)"/>
--->
+<!--   <xacro:planar_move prefix="$(arg prefix)"/> -->
    <xacro:agv prefix="$(arg prefix)"/>
    <!--<xacro:xtion_stand parent="agv_base_link" tilting_angle="0" /> -->

File: agv_low/urdf/sensors/asus_xtion_pro.urdf.xacro (robot description, xacro)
@@ -10,6 +10,15 @@
   <xacro:property name="M_PI" value="3.1415926535897931" />
   <xacro:macro name="sensor_asus_xtion_pro" params="prefix parent *origin">
+<!--    <link name="agv_base_link">
+	<visual>
+		<origin xyz="0 0 0" rpy="0 0 0" />
+		<geometry>
+			<box size="0.001 0.001 0.001" />
+		</geometry>
+	</visual>
+    </link>
+-->
     <joint name="${prefix}_rgb_joint" type="fixed">
-      <xacro:insert_block name="origin" />
+	  <xacro:insert_block name="origin" />
       <parent link="${parent}"/>
       <child link="${prefix}_rgb_base_link" />
@@ -38,5 +47,5 @@
       </inertial>
     </link>
-    <joint name="${prefix}_joint" type="fixed">
+    <joint name="${prefix}_joint" type="fixed"> <!-- ${asus_xtion_pro_rgb_rel_rgb_py} visual x -0.01 -->
       <origin xyz="0 ${asus_xtion_pro_rgb_rel_rgb_py} 0"
               rpy="0 0 0"/>
@@ -46,13 +55,11 @@
     <link name="${prefix}_link">
       <visual>
-        <!--<origin xyz="-0.09 0.020715 0.0164" rpy="${-M_PI/2} -${M_PI} ${-M_PI/2}"/> -->
-	<origin xyz="0.0164 -0.068 0.020715" rpy="${-M_PI/2} -${M_PI} ${-M_PI/2}"/>
+        <origin xyz="-0.01 0 0" rpy="${-M_PI/2} -${M_PI} ${-M_PI/2}"/>
         <geometry>
-          <mesh filename="package://agv_low/meshes/sensors/asus_xtion_pro_new.dae" scale="${asus_xtion_scale} ${asus_xtion_scale} ${asus_xtion_scale}"/>
+          <mesh filename="package://agv_low/meshes/sensors/asus_xtion_pro_live.dae" scale="${asus_xtion_scale} ${asus_xtion_scale} ${asus_xtion_scale}"/>
         </geometry>
       </visual>
       <collision>
-        <!-- <origin xyz="-0.090 0.020715 0.016400" rpy="0 0 0" /> -->
-	<origin xyz="0.0164 -0.068 0.020715" rpy="0 0 0" />
+        <origin xyz="0.0 0.0 0.0" rpy="0 0 0" />
         <geometry>
         <box size="0.0730 .2760 0.0720"/>
@@ -67,5 +74,5 @@
       </inertial>
     </link>
-    <joint name="${prefix}_depth_joint" type="fixed">
+    <joint name="${prefix}_depth_joint" type="fixed"> <!-- y ${asus_xtion_pro_depth_rel_rgb_py} -->
       <origin xyz="0 ${asus_xtion_pro_depth_rel_rgb_py} 0" rpy="0 0 0" />
       <parent link="${prefix}_rgb_base_link" />
@@ -96,5 +103,5 @@
     </link>
   <!-- RGBD sensor for simulation, same as Kinect -->
-  <sensor_xtion_pro_gazebo />
+  <sensor_xtion_pro_gazebo/>
   </xacro:macro>
    <xacro:macro name="sensor_xtion_pro_gazebo">

Commit message: added new mesh files with reduced faces and used in urdf

File: agv_low/robots/agv_urdf_youbot_collsionwheel.xacro (robot description, xacro)
@@ -34,5 +34,4 @@
   		<xacro:mecanum_wheel_visual prefix="${prefix}back_right" angle="1" wheel_pos="1" parent="${prefix}base_link" />
   		<!-- IMU -->
-<!--
 		<xacro:sensor_imu_hector prefix="$(arg prefix)imu" parent="$(arg prefix)base_link">
 			<origin xyz="0.48 0.0 0.338" rpy="0 0 0"/>
@@ -44,13 +43,12 @@
 			<origin xyz="0.060 -0.349 0.338" rpy="0 0 3.1416"/>
 		</xacro:sensor_sick_s300>
-		<xacro:sensor_asus_xtion_pro prefix="$(arg prefix)xtion" parent="$(arg prefix)base_link" > -->
+		<xacro:sensor_asus_xtion_pro prefix="$(arg prefix)xtion" parent="$(arg prefix)base_link" >
 			<!--<origin xyz="0.900 -0.0235 0.338" rpy="0 0 0" /> -->
-<!--			<origin xyz="0.87852 -0.0015 0.36875" rpy="0 -1.571 0" />
+			<origin xyz="0.87852 -0.0015 0.36875" rpy="0 -1.571 0" />
 		</xacro:sensor_asus_xtion_pro>
 		<xacro:sensor_asus_xtion_pro_stand prefix="$(arg prefix)xtion_stand" parent="$(arg prefix)base_link" > -->
 			<!--<origin xyz="0.900 -0.0235 0.338" rpy="0 0 0" /> -->
-<!--			<origin xyz="0.900 -0.0235 0.338" rpy="0 0 0" />
+			<origin xyz="0.900 -0.0235 0.338" rpy="0 0 0" />
 		</xacro:sensor_asus_xtion_pro_stand>
--->
    	</xacro:macro>
    <!-- Gazebo ros control pluggins -->

File: agv_low/urdf/wheels/agv_low_wheel_urdf_visualwheel.xacro (robot description, xacro)
@@ -1,5 +1,5 @@
 <?xml version="1.0" encoding="UTF-8"?>
 <robot name="wheel" xmlns:xacro="http://www.ros.org/wiki/xacro">
-  <xacro:property name="wheel_mass" value="0.1" /> <!-- 2.166 in kg-->
+  <xacro:property name="wheel_mass" value="2.166" /> <!-- 2.166 in kg-->
   <xacro:property name="pi" value="3.14159"/>
   <xacro:macro name="mecanum_inertia">
@@ -33,10 +33,10 @@
           <xacro:if value="${wheel_pos}">
             <geometry>
-              <mesh filename="package://agv_low/meshes/Radbefestigung mit Motor-Getrieb (LVA33)_wheels.stl" />
+              <mesh filename="package://agv_low/meshes/Radbefestigung mit Motor-Getrieb (LVA33)_wheels_simplified_mesh.stl" />
             </geometry>
           </xacro:if>
           <xacro:unless value="${wheel_pos}">
             <geometry>
-              <mesh filename="package://agv_low/meshes/Radbefestigung mit Motor-Getrieb (LVA33)_MIR_wheels.stl" />
+              <mesh filename="package://agv_low/meshes/Radbefestigung mit Motor-Getrieb (LVA33)_MIR_wheels_simplified_mesh.stl" />
             </geometry>
 	  </xacro:unless>

Commit message: altered the mass and inertia of visual mecanum wheel

File: agv_low/robots/agv_urdf_youbot_collsionwheel.xacro (robot description, xacro)
@@ -47,5 +47,5 @@
 			<origin xyz="0.87852 -0.0015 0.36875" rpy="0 -1.571 0" />
 		</xacro:sensor_asus_xtion_pro>
-		<xacro:sensor_asus_xtion_pro_stand prefix="$(arg prefix)xtion_stand" parent="$(arg prefix)base_link" > -->
+		<xacro:sensor_asus_xtion_pro_stand prefix="$(arg prefix)xtion_stand" parent="$(arg prefix)base_link" >
 			<!--<origin xyz="0.900 -0.0235 0.338" rpy="0 0 0" /> -->
 			<origin xyz="0.900 -0.0235 0.338" rpy="0 0 0" />

File: agv_low/urdf/wheels/agv_low_wheel_urdf_visualwheel.xacro (robot description, xacro)
@@ -1,10 +1,10 @@
 <?xml version="1.0" encoding="UTF-8"?>
 <robot name="wheel" xmlns:xacro="http://www.ros.org/wiki/xacro">
-  <xacro:property name="wheel_mass" value="2.166" /> <!-- 2.166 in kg-->
+  <xacro:property name="wheel_mass" value="0.6" /> <!-- 2.166 in kg-->
   <xacro:property name="pi" value="3.14159"/>
   <xacro:macro name="mecanum_inertia">
-    <inertia  ixx="0.000" ixy = "0" ixz = "0"
-              iyy="0.000" iyz = "0"
-              izz="0.000" />
+    <inertia  ixx="1.5" ixy = "0" ixz = "0"
+              iyy="1.5" iyz = "0"
+              izz="1.5" />
   </xacro:macro>
   <xacro:macro name="mecanum_wheel_visual" params="prefix angle wheel_pos parent">

Commit message: updated the sensors positions

File: agv_low/robots/agv_urdf_youbot_collsionwheel.xacro (robot description, xacro)
@@ -36,5 +36,4 @@
 		<!-- Gazebo ros control pluggins -->
   		<!-- IMU -->
-<!--
 		<xacro:sensor_imu_hector prefix="$(arg prefix)imu" parent="$(arg prefix)base_link">
 			<origin xyz="0.0 0.0 0.0" rpy="0 0 0"/>
@@ -48,11 +47,11 @@
 		<xacro:sensor_asus_xtion_pro prefix="$(arg prefix)xtion" parent="$(arg prefix)base_link" > -->
 			<!--<origin xyz="0.900 -0.0235 0.338" rpy="0 0 0" /> -->
-<!--			<origin xyz="0.39852 -0.0015 0.36875" rpy="0 -1.571 0" />
+ 			<!--<origin xyz="0.87852 -0.0015 0.36875" rpy="0 -1.571 0" /> -->
+			<origin xyz="0.39852 -0.0015 0.03075" rpy="0 -1.571 0" /> <!-- "0.39852 -0.0015 0.36875" rpy="0 -1.571 0" -->
 		</xacro:sensor_asus_xtion_pro>
 		<xacro:sensor_asus_xtion_pro_stand prefix="$(arg prefix)xtion_stand" parent="$(arg prefix)base_link" > -->
 			<!--<origin xyz="0.900 -0.0235 0.338" rpy="0 0 0" /> -->
-<!--			<origin xyz="0.42 -0.0235 0.0" rpy="0 0 0" />
+			<origin xyz="0.42 -0.0235 0.0" rpy="0 0 0" />
 		</xacro:sensor_asus_xtion_pro_stand>
--->
    	</xacro:macro>
    <!-- Gazebo ros control pluggins -->
